Commit message: Fixes: - fixes mqtt library in cmakelists - adds dependencies to package.xml - changes urdf to match real robot

File: description/robot_core.xacro (robot description, xacro)
@@ -2,6 +2,6 @@
 <robot xmlns:xacro="http://www.ros.org/wiki/xacro" >
     <xacro:include filename="inertial_macros.xacro"/>
-    <xacro:property name="chassis_length" value="0.335"/>
-    <xacro:property name="chassis_width" value="0.265"/>
+    <xacro:property name="chassis_length" value="0.39"/>
+    <xacro:property name="chassis_width" value="0.3"/>
     <xacro:property name="chassis_radius" value="0.15"/>
     <xacro:property name="chassis_height" value="0.075"/>
@@ -49,5 +49,5 @@
         <origin xyz="-0.1 0 0"/>
     </joint>
-    <!-- <link name="chassis">
+    <link name="chassis">
         <visual>
             <origin xyz="${chassis_length/2} 0 ${chassis_height/2}"/>
@@ -66,6 +66,6 @@
             <origin xyz="${chassis_length/2} 0 ${chassis_height/2}" rpy="0 0 0"/>
         </xacro:inertial_box>
-    </link> -->
-    <link name="chassis">
+    </link>
+    <!-- <link name="chassis">
         <visual>
             <origin xyz="0.15 0 0.075"/>
@@ -84,5 +84,5 @@
             <origin xyz="0.15 0 0.075" rpy="0 0 0" />
         </xacro:inertial_cylinder>
-    </link>
+    </link> -->
     <gazebo reference="chassis">
         <material>Gazebo/Orange</material>

Commit message: Adjusts robot's shape and nav2 parameters for smoother navigation

File: description/robot_core.xacro (robot description, xacro)
@@ -92,5 +92,5 @@
         <parent link="base_link"/>
         <child link="left_wheel"/>
-        <origin xyz="-0.065 ${wheel_offset_y} 0" rpy="-${pi/2} 0 0" />
+        <origin xyz="0 ${wheel_offset_y} 0" rpy="-${pi/2} 0 0" />
         <axis xyz="0 0 1"/>
     </joint>
@@ -118,5 +118,5 @@
         <parent link="base_link"/>
         <child link="right_wheel"/>
-        <origin xyz="-0.065 ${-wheel_offset_y} 0" rpy="${pi/2} 0 0" />
+        <origin xyz="0 ${-wheel_offset_y} 0" rpy="${pi/2} 0 0" />
         <axis xyz="0 0 -1"/>
     </joint>
